Commit message: camera position changed

File: src/ROV_model_URDF/urdf/ROV_model_URDF.xacro (robot description, xacro)
@@ -553,5 +553,5 @@
   <link name="camera_front_left">
     <visual>
-      <origin xyz="0.05 -0.08 -0.03" rpy="-1.5708 0 0"/>
+      <origin xyz="0.05 -0.08 -0.0" rpy="-1.5708 0 0"/>
       <geometry>
         <box size="${cameraSize} ${cameraSize} ${cameraSize}"/>
